File: Electrical/Detector2.sch (KiCad schematic (older format))
At the start: 0 parts

Commit message: Added placeholder for other sheets in schematic. Added peltier supply regulator and analog supply regulator.
Other:
- note removed: "Capacitors - 16V X5R\nResistors - 1/10W 10%"
- note removed: "Unlabelled Components:"
Changed lines of the file:
@@
 $Descr A4 11700 8267
 encoding utf-8
-Sheet 1 5
+Sheet 3 5
 Title "Cosmic Ray Detector"
 Date "16 apr 2013"
@@
 Comment4 ""
 $EndDescr
-$Sheet
-S 6100 3450 1000 1000
-U 516B8E64
-F0 "Power" 60
-F1 "Power.sch" 60
-$EndSheet
-$Sheet
-S 3100 4200 1000 1000
-U 516B8E0E
-F0 "Detector2" 60
-F1 "Detector2.sch" 60
-$EndSheet
-$Sheet
-S 3100 2700 1000 1000
-U 516B74CB
-F0 "Detector1" 60
-F1 "Detector1.sch" 60
-$EndSheet
-$Sheet
-S 4600 3450 1000 1000
-U 516B5437
-F0 "Cooler" 60
-F1 "PeltierCooler.sch" 60
-$EndSheet
-Text Notes 9900 6400 0    60   ~ 12
-Unlabelled Components:
-Text Notes 9900 6500 0    60   ~ 0
-Capacitors - 16V X5R\nResistors - 1/10W 10%
 $EndSCHEMATC
