File: Electrical/Detector2.sch (KiCad schematic (older format))
At the start: 0 parts

Commit message: Added sensors/data logger with ChipKit Max
Parts:
- added C? (x3): 0.1uF, symbol C
- added C? (x2): 0.15uF, symbol C
- added C? (x2): 1uF, symbol C
- added C?: 4.7uF, symbol C
- added C? (x2): 0.01uF, symbol C
- added C?: 100pF, symbol C
- added C? (x2): C, symbol C
- added D? (x5): MBR0540, symbol DIODESCH
- added D?: uFB10035-X18, symbol PHOTODIODE
- added FB? (x2): FERRITE, symbol FERRITE
- added L?: INDUCTOR, symbol INDUCTOR
- added R? (x10): R, symbol R
- added TP?: TP_Det, symbol CONN_4
- added U?: LT1930, symbol LT1930
- added U?: OPA380, symbol OPA381
Connections:
- new net: C?.2, R?.1, R?.2, R?.2, R?.2
- new net: C?.1, C?.1, D?.2 (K), R?.1, R?.1
- new net: D?.2 (K), R?.1, U?.3 (FB)
- new net: C?.2, D?.1 (A), D?.2 (K), L?.2, U?.1 (SW)
- new net: C?.1, C?.2, D?.1 (A), D?.2 (K)
- new net: C?.1, D?.1 (A), D?.2 (K)
- new net: R?.2, U?.4 (~Shdn)
- new net: C?.1, C?.1, D?.1, R?.1, U?.2 (-)
- new net: C?.1, R?.1, U?.3 (+)
- new net: C?.2, R?.1, R?.2, U?.6
- new net: C?.1, C?.1, FB?.2, U?.7
- new net: C?.1, C?.1, D?.2, FB?.2
- new net +5VA: FB?.1
- new net +BATT: C?.1, L?.1, R?.1, U?.5 (VIn)
- new net BiasSet: R?.1
- new net Det: R?.2, TP?.2 (P2)
- new net GND: C?.2, C?.2, C?.2, C?.2, C?.2, C?.2, C?.2, C?.2, C?.2, D?.1 (A), D?.1 (A), R?.2, R?.2, R?.2, TP?.4 (P4), U?.2 (Gnd), U?.4
- new net HS: D?.3, TP?.3 (P3)
- new net VBias: C?.1, FB?.1, R?.1, R?.2, TP?.1 (P1)
Other:
- note added: "Bias Supply"
- note added: "Detector/Amplifier"
- note added: "Fast Mode Output"
- note added: "Fiber Optic\nDevice Mount"
- note added: "Optional:\nOmit if not using fast mode"
- note added: "Power Supply"
- note added: "Standard Output"

Commit message: Annotated schematic
Parts:
- gave numbers to parts that had none: 35
