File: Electrical/Sensors.sch (KiCad schematic (older format))
At the start: 21 parts

Commit message: Annotated schematic
Parts:
- added unit 5 of J2
- added unit 6 of J2
- added R4, R5: R, symbol R
- gave numbers to parts that had none: 19
Connections:
- wire segments 110 -> 90
- no-connect marks 18 -> 70
Other:
- moved on the sheet: C7, J2H, J2I, J2J
